File: 01_cad/carChargeChannel.brd (EAGLE design)
At the start: 100.3 x 80 mm, 126 parts, among them IC1 LT1513, IC2 PIC18F2420, IC3 TPS60403, IC4 7805, T1 BC847A, T2 IRL530, T3 BSS138, T4 BSS138, X2 2X3, X3 DIN5

Commit message: ongoing...
Parts:
- added C38: 4µ7, omcCapacitor:1206
- added C39: 100n/50V, omcCapacitor:1206
- C7: device omcCapacitor:0805 -> omcCapacitor:1206
- L1, L2: device omcInductor:PIS472X -> omcInductor:DR74
- moved C2 137.3 mm to (24.1, 17.8), turned to 90 degrees
- moved L1 133.7 mm to (27.3, 38.1), turned to 270 degrees
- moved T1 123.5 mm to (26.0, 5.08), turned to 90 degrees
- moved T2 120.0 mm to (26.7, 61.0)
- moved C1 119.0 mm to (17.8, 29.8), turned to 90 degrees
- moved D4 118.0 mm to (33.7, 5.08), turned to 270 degrees
- moved R3 114.0 mm to (14.6, 10.8), turned to 90 degrees
- moved R5 110.8 mm to (30.5, 5.08), turned to 90 degrees
- moved R25 107.2 mm to (24.1, 10.8), turned to 270 degrees
- moved R4 104.4 mm to (33.7, 10.8), turned to 90 degrees
- moved R22 103.4 mm to (30.5, 10.8), turned to 90 degrees
- moved R24 101.6 mm to (21.0, 10.8), turned to 270 degrees
- moved R2 97.7 mm to (17.8, 35.6), turned to 270 degrees
- moved IC1 96.9 mm to (8.89, 20.3), turned to 90 degrees
- moved R21 89.0 mm to (21.0, 17.8), turned to 270 degrees
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Connections:
- net GND: now also C39.2
- net N$1: now also C38.2
- net N$2: now also C38.1
- net VBAT: now also C39.1
Routing:
- net N$9: track 0.00 -> 29.9 mm, vias 0 -> 2
- net N$2: track 0.00 -> 8.21 mm
- net N$8: track 0.00 -> 7.89 mm
- net N$7: track 0.00 -> 4.88 mm
- net N$6: track 0.00 -> 4.34 mm
- added copper zone on layer 1, net GND
- added copper zone on layer 16, net GND

Commit message: intermediate
Parts:
- added C40: 47µ/16V, omcCapacitor:1210
- added C41: 47µ/6V, omcCapacitor:1206
- C28: value 10µ/16V -> 100n/50V
- C31: value 47µ/16V -> 47µ/6V; device omcCapacitor:PANC -> omcCapacitor:1206
- C45: value 10µ/16V -> 47µ/16V; device omcCapacitor:1206 -> omcCapacitor:1210
- C5: value 100µ/6V -> 47µ/6V
- D2: value PMEG2010 -> BAT46; device omcDiode:SOD323 -> omcDiode:SOD123
- moved C44 162.6 mm to (67.3, 69.2), turned to 180 degrees
- moved R7 156.4 mm to (58.4, 17.8), turned to 90 degrees
- moved IC3 150.9 mm to (67.3, 64.8), turned to 180 degrees
- moved C43 148.6 mm to (62.2, 67.9), turned to 90 degrees
- moved C28 145.4 mm to (41.3, 62.2), turned to 90 degrees
- moved C42 145.1 mm to (67.3, 61.0), turned to 180 degrees
- moved C20 130.2 mm to (23.5, 55.9), turned to 180 degrees
- moved LED1 128.3 mm to (88.9, 62.2)
- moved X2 127.3 mm to (69.8, 75.6), turned to 90 degrees
- moved IC2 126.7 mm to (86.4, 45.7), turned to 270 degrees
- moved R33 125.4 mm to (73.7, 53.3), turned to 90 degrees
- moved OPA1 119.8 mm to (41.9, 50.8), turned to 270 degrees
- moved D2 119.3 mm to (23.5, 49.5)
- moved IC4 117.2 mm to (49.5, 68.6)
- moved C48 115.7 mm to (71.1, 6.35)
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Connections:
- net +12V: now also C40.1; no longer C31.CP, C47.1
- net EN_XCHRG: now also IC2.23
- net GND: now also C40.2, C41.2; no longer C31.CN
- net VCC: now also C41.1, C47.1
Routing:
- net N$23: track 0.00 -> 15.4 mm
- net N$26: track 0.00 -> 7.01 mm
- net N$22: track 0.00 -> 6.45 mm
- net N$21: track 0.00 -> 3.18 mm
- net N$25: track 0.00 -> 3.18 mm
- net N$28: track 0.00 -> 2.57 mm
- added copper zone on layer 1, net VBAT
- added copper zone on layer 16, net VBAT

Commit message: ongoing...
Parts:
- C13, C14, C15: value 100n -> 100n/50V; device omcCapacitor:0805 -> omcCapacitor:1206
- moved C17 163.1 mm to (88.9, 50.8)
- moved R17 156.9 mm to (59.1, 48.9), turned to 180 degrees
- moved R29 152.2 mm to (86.4, 57.1)
- moved R15 150.8 mm to (45.7, 43.8)
- moved C24 149.9 mm to (81.3, 64.8)
- moved L5 147.9 mm to (76.2, 67.3), turned to 270 degrees
- moved C25 141.7 mm to (82.5, 68.6)
- moved C23 141.2 mm to (81.3, 62.2)
- moved L4 137.7 mm to (72.4, 67.3), turned to 270 degrees
- moved R14 134.9 mm to (45.7, 40.0), turned to 180 degrees
- moved C15 133.2 mm to (45.7, 51.4), turned to 180 degrees
- moved R16 130.2 mm to (40.3, 59.1)
- moved R10 127.8 mm to (28.6, 40.0)
- moved R18 127.5 mm to (22.9, 51.4), turned to 180 degrees
- moved R13 122.3 mm to (40.0, 43.8), turned to 180 degrees
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Routing:
- net N$11: track 0.00 -> 16.1 mm
- net N$21: track 3.18 -> 15.9 mm
- net -5V: track 0.00 -> 11.7 mm
- net N$15: track 0.00 -> 11.4 mm
- net +5V: track 0.00 -> 11.2 mm
- net N$24: track 0.00 -> 11.1 mm
- net N$12: track 0.00 -> 10.9 mm
- net N$17: track 0.00 -> 8.84 mm
- net N$3: track 0.00 -> 8.39 mm
- net GNDA: track 0.00 -> 8.13 mm, vias 0 -> 4
- net N$13: track 0.00 -> 8.05 mm
- net N$25: track 3.18 -> 10.4 mm
- net IM_CHG: track 0.00 -> 6.90 mm
- net N$23: track 15.4 -> 8.90 mm
- net EN_XCHRG: track 0.00 -> 6.11 mm, vias 0 -> 1
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
Commit message: ongoing...
Parts:
- removed C31: 47µ/6V, omcCapacitor:1206
- moved R39 181.2 mm to (58.4, 17.8)
- moved C21 176.4 mm to (81.3, 43.8), turned to 180 degrees
- moved C22 172.5 mm to (62.9, 30.5), turned to 90 degrees
- moved C19 166.8 mm to (81.3, 40.0), turned to 180 degrees
- moved R19 164.4 mm to (55.9, 57.1), turned to 180 degrees
- moved DAC2 163.2 mm to (61.0, 38.1)
- moved DAC1 159.4 mm to (66.0, 38.1)
- moved R36 158.6 mm to (52.1, 17.8)
- moved R37 158.0 mm to (45.7, 19.1)
- moved R6 149.5 mm to (49.5, 14.0)
- moved OSC1 144.1 mm to (59.7, 27.9), turned to 90 degrees
- moved C18 141.0 mm to (45.7, 59.1), turned to 180 degrees
- moved C32 135.7 mm to (59.7, 5.08), turned to 90 degrees
- moved REF1 127.0 mm to (76.2, 47.6), turned to 180 degrees
- moved R41 124.5 mm to (45.7, 22.9)
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Connections:
- net GND: no longer C18.1
- net GNDA: now also C18.1
Routing:
- net VREF_ADC: track 0.00 -> 22.7 mm
- net IS_XCHRG: track 0.00 -> 15.5 mm, vias 0 -> 1
- net VBAT: track 0.00 -> 14.5 mm
- net VCC: track 0.00 -> 12.4 mm
- net N$34: track 0.00 -> 11.3 mm
- net -5V: track 11.7 -> 22.9 mm
- net +5V: track 11.2 -> 22.0 mm
- net N$35: track 0.00 -> 9.24 mm
- net GNDA: track 8.13 -> 12.5 mm, vias 4 -> 10
- net N$26: track 5.78 -> 9.31 mm
- net N$16: track 0.00 -> 2.56 mm
- net N$25: track 10.4 -> 12.6 mm
- net N$23: track 8.90 -> 8.08 mm
- added copper zone on layer 16, net GNDA

Commit message: ongoing...
Parts:
- added D7: BAT46, omcDiode:SOD123
- moved R35 153.6 mm to (56.5, 24.8), turned to 180 degrees
- moved R34 153.1 mm to (62.2, 24.8), turned to 180 degrees
- moved C30 133.9 mm to (73.7, 21.0), turned to 180 degrees
- moved C29 125.3 mm to (73.7, 24.8), turned to 180 degrees
- moved R36 53.6 mm to (97.8, 45.7)
- moved R37 52.3 mm to (91.4, 44.5)
- moved R41 50.6 mm to (95.2, 33.0)
- moved R40 49.5 mm to (95.2, 27.9)
- moved R39 49.5 mm to (95.2, 50.8)
- moved R6 46.8 mm to (95.2, 24.1)
- moved C37 31.2 mm to (56.5, 28.6)
- moved REF1 28.1 mm to (67.3, 21.0), turned to 0 degrees
- moved OSC1 27.3 mm to (83.8, 40.6), turned to 270 degrees
- moved C35 27.0 mm to (80.6, 44.5), turned to 90 degrees
- moved C17 25.1 mm to (56.5, 32.4)
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Connections:
- removed net N$30: DAC1.5, DAC2.5, IC2.13, R36.1
- removed net VSS: DAC1.7, DAC2.7
- new net N$37: DAC1.5, DAC2.5, IC2.11, R36.1
- net GND: no longer C10.2, C33.2
- net GNDA: now also C10.2, C33.2, DAC1.7, DAC2.7
- net N$20: now also IC2.13; no longer IC2.11
- net VDD: now also D7.C
- net VOPA_AD: now also IC2.4; no longer IC2.5
- net VP12_AD: now also D7.A, IC2.5; no longer IC2.4
Routing:
- net VBAT_AD: track 0.00 -> 26.8 mm, vias 0 -> 2
- net IM_CHG_AD: track 0.00 -> 19.1 mm
- net VP12_AD: track 0.00 -> 17.2 mm
- net N$37: track 0.00 -> 10.7 mm
- net N$10: track 0.00 -> 10.2 mm
- net !MCLR: track 0.00 -> 5.30 mm, vias 0 -> 2
- net VREF_ADC: track 22.7 -> 19.0 mm
- net VCC: track 12.4 -> 13.6 mm
- net GNDA: vias 10 -> 14

Commit message: ongoging
Parts:
- removed C32: 100n, omcCapacitor:1206
- moved D6 199.6 mm to (86.4, 50.8)
- moved D5 187.9 mm to (86.4, 53.3)
- moved R50 153.8 mm to (78.7, 53.3)
- moved R49 140.6 mm to (71.1, 53.3)
- moved C10 129.1 mm to (68.6, 21.0), turned to 180 degrees
- moved C34 108.8 mm to (68.6, 24.8), turned to 180 degrees
- moved C33 103.3 mm to (68.6, 17.1), turned to 180 degrees
- moved C11 45.8 mm to (67.3, 50.8), turned to 0 degrees
- moved R39 33.9 mm to (61.6, 54.6)
- moved R37 30.5 mm to (61.6, 50.8)
- moved R40 23.6 mm to (74.3, 17.1), turned to 180 degrees
- moved R41 22.5 mm to (74.3, 24.8), turned to 180 degrees
- moved R6 21.2 mm to (74.3, 21.0), turned to 180 degrees
- moved C19 11.4 mm to (51.4, 28.6), turned to 180 degrees
- moved C29 9.92 mm to (80.0, 17.1)
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Connections:
- net GND: no longer C32.2
- net N$29: now also DAC2.6; no longer DAC2.8
- net N$31: now also DAC2.8; no longer DAC2.6
- net VDD: no longer C32.1
Routing:
- net !CS_DAC1: track 0.00 -> 29.2 mm, vias 0 -> 2
- net !CS_DAC2: track 0.00 -> 26.4 mm, vias 0 -> 2
- net N$20: track 0.00 -> 23.7 mm
- net VOPA_AD: track 0.00 -> 16.0 mm
- net GNDA: track 12.5 -> 27.6 mm, vias 14 -> 16
- net +5V: track 22.0 -> 36.4 mm
- net N$35: track 9.24 -> 18.9 mm
- net N$37: track 10.7 -> 18.7 mm, vias 0 -> 1
- net IM_CHG_AD: track 19.1 -> 14.0 mm
- net N$32: track 0.00 -> 3.68 mm
- net N$31: track 0.00 -> 3.68 mm
- net N$34: track 11.3 -> 14.3 mm
- net N$29: track 0.00 -> 2.40 mm
- net N$10: track 10.2 -> 11.9 mm
- net VBAT_AD: track 26.8 -> 25.5 mm

Commit message: intermediate
Parts:
- moved D3 94.8 mm to (43.2, 34.3)
- moved D7 30.7 mm to (55.9, 50.8), turned to 180 degrees
Connections:
- net N$10: now also IC2.13; no longer IC2.12
- net N$20: now also IC2.12; no longer IC2.13
Routing:
- net !CS_DAC2: track 26.4 -> 51.0 mm, vias 2 -> 4
- net N$10: track 11.9 -> 29.4 mm
- net !CS_DAC1: track 29.2 -> 41.7 mm
- net N$37: track 18.7 -> 29.8 mm, vias 1 -> 0
- net VP12_AD: track 17.2 -> 25.6 mm
- net N$20: track 23.7 -> 31.3 mm
- net VDD: track 0.00 -> 4.78 mm
- net VOPA_AD: track 16.0 -> 14.7 mm
- net !MCLR: track 5.30 -> 6.57 mm
- net GNDA: track 27.6 -> 27.1 mm, vias 16 -> 17
