File: 01_cad/carChargeChannel.sch (EAGLE design)
At the start: 130 parts, among them IC1 LT1513, IC2 PIC18F2420, IC3 TPS60403, IC4 7805, T1 BC847A, T2 IRL530, T3 BSS138, T4 BSS138, X2 2X3, X3 DIN5

Commit message: ongoing...
Parts:
- C13, C14, C15: value 100n -> 100n/50V; device omcCapacitor:X7R-100000P-0805 -> omcCapacitor:X7R-100000P-1206
Other:
- moved on the sheet: C13, C14
Changed lines of the file:
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@@
 <part name="FRAME2" library="frames" deviceset="A4L-LOC" device=""/>
 <part name="OPA1" library="omcOpAmp" deviceset="MCP6H04" device="" value="MCP6H04"/>
-<part name="C13" library="omcCapacitor" deviceset="X7R" device="-0805" technology="-100000P" value="100n"/>
-<part name="C14" library="omcCapacitor" deviceset="X7R" device="-0805" technology="-100000P" value="100n"/>
-<part name="C15" library="omcCapacitor" deviceset="X7R" device="-0805" technology="-100000P" value="100n"/>
+<part name="C13" library="omcCapacitor" deviceset="X7R" device="-1206" technology="-100000P" value="100n/50V"/>
+<part name="C14" library="omcCapacitor" deviceset="X7R" device="-1206" technology="-100000P" value="100n/50V"/>
+<part name="C15" library="omcCapacitor" deviceset="X7R" device="-1206" technology="-100000P" value="100n/50V"/>
 <part name="P+4" library="supply1" deviceset="+5V" device=""/>
 <part name="P-2" library="supply1" deviceset="-5V" device=""/>
@@
 </instance>
 <instance part="OPA1" gate="G$5" x="190.5" y="40.64"/>
-<instance part="C13" gate="G$1" x="172.72" y="45.72"/>
-<instance part="C14" gate="G$1" x="172.72" y="38.1"/>
+<instance part="C13" gate="G$1" x="167.64" y="45.72"/>
+<instance part="C14" gate="G$1" x="167.64" y="38.1"/>
 <instance part="C15" gate="G$1" x="182.88" y="43.18"/>
-<instance part="P+4" gate="1" x="165.1" y="48.26" smashed="yes" rot="R90">
-<attribute name="VALUE" x="163.83" y="49.276" size="1.778" layer="96" rot="R180"/>
-</instance>
-<instance part="P-2" gate="1" x="165.1" y="33.02" smashed="yes" rot="R270">
-<attribute name="VALUE" x="160.02" y="32.258" size="1.778" layer="96"/>
+<instance part="P+4" gate="1" x="160.02" y="48.26" smashed="yes" rot="R90">
+<attribute name="VALUE" x="158.75" y="49.276" size="1.778" layer="96" rot="R180"/>
+</instance>
+<instance part="P-2" gate="1" x="160.02" y="33.02" smashed="yes" rot="R270">
+<attribute name="VALUE" x="154.94" y="32.258" size="1.778" layer="96"/>
 </instance>
 <instance part="R26" gate="G$1" x="93.98" y="25.4" smashed="yes" rot="R90">
@@
 <attribute name="VALUE" x="72.39" y="129.54" size="1.778" layer="96" rot="R180"/>
 </instance>
-<instance part="GND15" gate="1" x="165.1" y="40.64" smashed="yes" rot="R270">
-<attribute name="VALUE" x="157.226" y="39.878" size="1.778" layer="96"/>
+<instance part="GND15" gate="1" x="160.02" y="40.64" smashed="yes" rot="R270">
+<attribute name="VALUE" x="152.146" y="39.878" size="1.778" layer="96"/>
 </instance>
 <instance part="P+13" gate="1" x="27.94" y="157.48" rot="R90"/>
@@
 <pinref part="C13" gate="G$1" pin="1"/>
 <wire x1="190.5" y1="48.26" x2="182.88" y2="48.26" width="0.1524" layer="91"/>
-<wire x1="182.88" y1="48.26" x2="172.72" y2="48.26" width="0.1524" layer="91"/>
-<wire x1="172.72" y1="48.26" x2="167.64" y2="48.26" width="0.1524" layer="91"/>
-<junction x="172.72" y="48.26"/>
+<wire x1="182.88" y1="48.26" x2="167.64" y2="48.26" width="0.1524" layer="91"/>
+<wire x1="167.64" y1="48.26" x2="162.56" y2="48.26" width="0.1524" layer="91"/>
+<junction x="167.64" y="48.26"/>
 <pinref part="P+4" gate="1" pin="+5V"/>
 <pinref part="C15" gate="G$1" pin="1"/>
@@
 <pinref part="C14" gate="G$1" pin="2"/>
 <wire x1="190.5" y1="33.02" x2="182.88" y2="33.02" width="0.1524" layer="91"/>
-<wire x1="182.88" y1="33.02" x2="172.72" y2="33.02" width="0.1524" layer="91"/>
-<wire x1="172.72" y1="33.02" x2="167.64" y2="33.02" width="0.1524" layer="91"/>
-<junction x="172.72" y="33.02"/>
+<wire x1="182.88" y1="33.02" x2="167.64" y2="33.02" width="0.1524" layer="91"/>
+<wire x1="167.64" y1="33.02" x2="162.56" y2="33.02" width="0.1524" layer="91"/>
+<junction x="167.64" y="33.02"/>
 <pinref part="P-2" gate="1" pin="-5V"/>
 <pinref part="C15" gate="G$1" pin="2"/>
@@
 <pinref part="C14" gate="G$1" pin="1"/>
 <pinref part="C13" gate="G$1" pin="2"/>
-<junction x="172.72" y="40.64"/>
-<wire x1="167.64" y1="40.64" x2="172.72" y2="40.64" width="0.1524" layer="91"/>
+<junction x="167.64" y="40.64"/>
+<wire x1="162.56" y1="40.64" x2="167.64" y2="40.64" width="0.1524" layer="91"/>
 <pinref part="GND15" gate="1" pin="GNDA"/>
 </segment>

Commit message: ongoing...
Parts:
- removed C31: 47µ/6V, omcCapacitor:X5R-47000000P-1206
Connections:
- net GND: no longer C18.1
- net GNDA: now also C18.1
Changed lines of the file:
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@@
 <part name="R19" library="omcResistor" deviceset="R1206" device="-1%" technology="-1000" value="1K"/>
 <part name="C18" library="omcCapacitor" deviceset="X7R" device="-1206" technology="-100000P" value="100n/50V"/>
-<part name="GND24" library="supply1" deviceset="GND" device=""/>
 <part name="R20" library="omcResistor" deviceset="R1206" device="-1%" technology="-2200" value="2K2"/>
 <part name="R21" library="omcResistor" deviceset="R1206" device="-1%" technology="-12000" value="12K"/>
@@
 <part name="C40" library="omcCapacitor" deviceset="X5R" device="-1210" technology="-47000000P" value="47µ/16V"/>
 <part name="C45" library="omcCapacitor" deviceset="X5R" device="-1210" technology="-47000000P" value="47µ/16V"/>
-<part name="C31" library="omcCapacitor" deviceset="X5R" device="-1206" technology="-47000000P" value="47µ/6V"/>
 <part name="C5" library="omcCapacitor" deviceset="X5R" device="-1206" technology="-47000000P" value="47µ/6V"/>
 <part name="C41" library="omcCapacitor" deviceset="X5R" device="-1206" technology="-47000000P" value="47µ/6V"/>
@@
 <part name="GND58" library="supply1" deviceset="GND" device=""/>
 <part name="C28" library="omcCapacitor" deviceset="X7R" device="-1206" technology="-100000P" value="100n/50V"/>
+<part name="GND24" library="supply1" deviceset="GNDA" device=""/>
 </parts>
 <sheets>
@@
 <instance part="C40" gate="G$1" x="55.88" y="137.16"/>
 <instance part="C45" gate="G$1" x="68.58" y="137.16"/>
-<instance part="C31" gate="G$1" x="101.6" y="167.64"/>
 <instance part="C5" gate="G$1" x="134.62" y="137.16"/>
 <instance part="C41" gate="G$1" x="121.92" y="137.16"/>
@@
 <attribute name="VALUE" x="153.924" y="96.901" size="1.778" layer="96"/>
 </instance>
-<instance part="GND24" gate="1" x="152.4" y="93.98" rot="R270"/>
 <instance part="R20" gate="G$1" x="200.66" y="86.36"/>
 <instance part="OPA1" gate="G$4" x="58.42" y="38.1" smashed="yes">
@@
 <attribute name="VALUE" x="77.47" y="50.5206" size="1.778" layer="96"/>
 </instance>
+<instance part="GND24" gate="1" x="152.4" y="93.98" smashed="yes" rot="R270">
+<attribute name="VALUE" x="151.13" y="90.932" size="1.778" layer="96" rot="R90"/>
+</instance>
 </instances>
 <busses>
@@
 <wire x1="76.2" y1="129.54" x2="76.2" y2="121.92" width="0.1524" layer="91"/>
 <pinref part="T1" gate="G$1" pin="E"/>
-</segment>
-<segment>
-<pinref part="C18" gate="G$1" pin="1"/>
-<pinref part="GND24" gate="1" pin="GND"/>
 </segment>
 <segment>
@@
 <pinref part="GND15" gate="1" pin="GNDA"/>
 </segment>
-</net>
+<segment>
+<pinref part="C18" gate="G$1" pin="1"/>
+<pinref part="GND24" gate="1" pin="GNDA"/>
+</segment>
+</net>

Commit message: ongoing...
Parts:
- added D7: BAT46, omcDiode:BAT46W
Connections:
- removed net N$30: DAC1G$1.!LDAC, DAC2G$1.!LDAC, IC2.2@RC, R36.1
- removed net VSS: DAC1G$2.VSS, DAC2G$2.VSS
- new net N$37: DAC1G$1.!LDAC, DAC2G$1.!LDAC, IC2.0@RC, R36.1
- net GND: no longer C10.2, C33.2
- net GNDA: now also C10.2, C33.2, DAC1G$2.VSS, DAC2G$2.VSS
- net N$20: now also IC2.2@RC; no longer IC2.0@RC
- net VDD: now also D7.C
- net VOPA_AD: now also IC2.2@RA; no longer IC2.3@RA
- net VP12_AD: now also D7.A, IC2.3@RA; no longer IC2.2@RA
Other:
- moved on the sheet: C10, C33, C34, C37, D3, DAC1, DAC2, R36, R37, R39, R40, R41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

Commit message: ongoging
Parts:
- removed C32: 100n, omcCapacitor:X7R-100000P-1206
Connections:
- net GND: no longer C32.2
- net N$29: now also DAC2G$1.VOUTB; no longer DAC2G$1.VOUTA
- net N$31: now also DAC2G$1.VOUTA; no longer DAC2G$1.VOUTB
- net VDD: no longer C32.1
Other:
- moved on the sheet: C10, C12, C33, R40, R6
Changed lines of the file:
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@@
 <part name="C30" library="omcCapacitor" deviceset="X7R" device="-1206" technology="-100000P" value="100n"/>
 <part name="GND43" library="supply1" deviceset="GNDA" device=""/>
-<part name="C32" library="omcCapacitor" deviceset="X7R" device="-1206" technology="-100000P" value="100n"/>
 <part name="C10" library="omcCapacitor" deviceset="X7R" device="-1206" technology="-2200000P" value="2µ2/50V"/>
 <part name="R40" library="omcResistor" deviceset="RC1206" device="" technology="-470" value="470R"/>
@@
 <text x="91.694" y="87.376" size="1.4224" layer="98">CH = 25pF</text>
 <text x="187.96" y="160.02" size="1.9304" layer="98">starring point</text>
+<text x="200.66" y="73.66" size="1.4224" layer="98">Fc=153Hz</text>
 <text x="200.66" y="88.9" size="1.4224" layer="98">Fc=153Hz</text>
-<text x="200.66" y="73.66" size="1.4224" layer="98">Fc=153Hz</text>
 <text x="200.66" y="104.14" size="1.4224" layer="98">Fc=153Hz</text>
 <text x="43.18" y="55.88" size="1.6764" layer="98">caps close to
@@
 <instances>
 <instance part="FRAME1" gate="G$1" x="0" y="0"/>
-<instance part="R6" gate="G$1" x="205.74" y="93.98"/>
+<instance part="R6" gate="G$1" x="205.74" y="78.74"/>
 <instance part="C11" gate="G$1" x="101.6" y="66.04"/>
-<instance part="C12" gate="G$1" x="86.36" y="66.04"/>
+<instance part="C12" gate="G$1" x="93.98" y="66.04"/>
 <instance part="P+3" gate="1" x="223.52" y="167.64" rot="R270"/>
-<instance part="GND33" gate="1" x="86.36" y="55.88"/>
+<instance part="GND33" gate="1" x="93.98" y="55.88"/>
 <instance part="REF1" gate="G$1" x="76.2" y="81.28" smashed="yes" rot="R90">
 <attribute name="NAME" x="78.74" y="82.423" size="1.778" layer="95"/>
@@
 <attribute name="VALUE" x="12.192" y="10.16" size="1.778" layer="96"/>
 </instance>
-<instance part="C32" gate="G$1" x="93.98" y="66.04"/>
-<instance part="C10" gate="G$1" x="213.36" y="91.44"/>
-<instance part="R40" gate="G$1" x="205.74" y="78.74"/>
-<instance part="C33" gate="G$1" x="213.36" y="76.2"/>
+<instance part="C10" gate="G$1" x="213.36" y="76.2"/>
+<instance part="R40" gate="G$1" x="205.74" y="93.98"/>
+<instance part="C33" gate="G$1" x="213.36" y="91.44"/>
 <instance part="R41" gate="G$1" x="205.74" y="109.22"/>
 <instance part="C34" gate="G$1" x="213.36" y="106.68"/>
@@
 <instance part="GND58" gate="1" x="154.94" y="129.54"/>
 <instance part="C28" gate="G$1" x="81.28" y="137.16"/>
-<instance part="GND13" gate="1" x="213.36" y="83.82" smashed="yes">
+<instance part="GND13" gate="1" x="213.36" y="68.58" smashed="yes">
+<attribute name="VALUE" x="210.312" y="66.04" size="1.778" layer="96"/>
+</instance>
+<instance part="GND32" gate="1" x="213.36" y="83.82" smashed="yes">
 <attribute name="VALUE" x="210.312" y="81.28" size="1.778" layer="96"/>
-</instance>
-<instance part="GND32" gate="1" x="213.36" y="68.58" smashed="yes">
-<attribute name="VALUE" x="210.312" y="66.04" size="1.778" layer="96"/>
 </instance>
 <instance part="D7" gate="G$1" x="76.2" y="30.48" smashed="yes" rot="R90">
@@
 <pinref part="C11" gate="G$1" pin="2"/>
 <wire x1="101.6" y1="58.42" x2="101.6" y2="60.96" width="0.1524" layer="91"/>
+<junction x="101.6" y="58.42"/>
 <wire x1="101.6" y1="58.42" x2="93.98" y2="58.42" width="0.1524" layer="91"/>
-<junction x="101.6" y="58.42"/>
-<pinref part="C32" gate="G$1" pin="2"/>
+<pinref part="C12" gate="G$1" pin="2"/>
 <wire x1="93.98" y1="58.42" x2="93.98" y2="60.96" width="0.1524" layer="91"/>
-<wire x1="93.98" y1="58.42" x2="86.36" y2="58.42" width="0.1524" layer="91"/>
+<pinref part="GND33" gate="1" pin="GND"/>
 <junction x="93.98" y="58.42"/>
-<pinref part="C12" gate="G$1" pin="2"/>
-<wire x1="86.36" y1="58.42" x2="86.36" y2="60.96" width="0.1524" layer="91"/>
-<pinref part="GND33" gate="1" pin="GND"/>
-<junction x="86.36" y="58.42"/>
 <pinref part="IC2" gate="G$1" pin="VSS@VSS0"/>
 <pinref part="IC2" gate="G$1" pin="VSS@VSS1"/>
@@
 <segment>
 <pinref part="R6" gate="G$1" pin="2"/>
-<label x="213.868" y="94.488" size="1.778" layer="95"/>
-<wire x1="210.82" y1="93.98" x2="213.36" y2="93.98" width="0.1524" layer="91"/>
+<label x="213.868" y="79.248" size="1.778" layer="95"/>
+<wire x1="210.82" y1="78.74" x2="213.36" y2="78.74" width="0.1524" layer="91"/>
 <pinref part="C10" gate="G$1" pin="1"/>
-<wire x1="213.36" y1="93.98" x2="220.98" y2="93.98" width="0.1524" layer="91"/>
-<junction x="213.36" y="93.98"/>
+<wire x1="213.36" y1="78.74" x2="220.98" y2="78.74" width="0.1524" layer="91"/>
+<junction x="213.36" y="78.74"/>
 </segment>
 </net>
@@
 <segment>
 <pinref part="C11" gate="G$1" pin="1"/>
-<wire x1="86.36" y1="71.12" x2="93.98" y2="71.12" width="0.1524" layer="91"/>
 <wire x1="93.98" y1="71.12" x2="101.6" y2="71.12" width="0.1524" layer="91"/>
 <wire x1="101.6" y1="71.12" x2="109.22" y2="71.12" width="0.1524" layer="91"/>
 <wire x1="101.6" y1="68.58" x2="101.6" y2="71.12" width="0.1524" layer="91"/>
 <junction x="101.6" y="71.12"/>
-<pinref part="C32" gate="G$1" pin="1"/>
+<pinref part="C12" gate="G$1" pin="1"/>
 <wire x1="93.98" y1="68.58" x2="93.98" y2="71.12" width="0.1524" layer="91"/>
-<junction x="93.98" y="71.12"/>
-<pinref part="C12" gate="G$1" pin="1"/>
-<wire x1="86.36" y1="68.58" x2="86.36" y2="71.12" width="0.1524" layer="91"/>
 <pinref part="D5" gate="G$1" pin="C"/>
 <wire x1="66.04" y1="71.12" x2="81.28" y2="71.12" width="0.1524" layer="91"/>
-<junction x="86.36" y="71.12"/>
-<wire x1="81.28" y1="71.12" x2="86.36" y2="71.12" width="0.1524" layer="91"/>
+<junction x="93.98" y="71.12"/>
+<wire x1="81.28" y1="71.12" x2="93.98" y2="71.12" width="0.1524" layer="91"/>
 <wire x1="81.28" y1="71.12" x2="81.28" y2="58.42" width="0.1524" layer="91"/>
 <junction x="81.28" y="71.12"/>
@@
 <net name="VS_CHG" class="0">
 <segment>
-<label x="213.868" y="79.248" size="1.778" layer="95"/>
-<wire x1="223.52" y1="78.74" x2="213.36" y2="78.74" width="0.1524" layer="91"/>
+<label x="213.868" y="94.488" size="1.778" layer="95"/>
+<wire x1="223.52" y1="93.98" x2="213.36" y2="93.98" width="0.1524" layer="91"/>
 <pinref part="C33" gate="G$1" pin="1"/>
 <pinref part="R40" gate="G$1" pin="2"/>
-<wire x1="210.82" y1="78.74" x2="213.36" y2="78.74" width="0.1524" layer="91"/>
-<junction x="213.36" y="78.74"/>
+<wire x1="210.82" y1="93.98" x2="213.36" y2="93.98" width="0.1524" layer="91"/>
+<junction x="213.36" y="93.98"/>
 </segment>
 </net>
 <net name="N$29" class="0">
 <segment>
+<pinref part="R6" gate="G$1" pin="1"/>
+<wire x1="198.12" y1="78.74" x2="200.66" y2="78.74" width="0.1524" layer="91"/>
+<wire x1="198.12" y1="78.74" x2="198.12" y2="83.82" width="0.1524" layer="91"/>
+<pinref part="DAC2" gate="G$1" pin="VOUTB"/>
+<wire x1="198.12" y1="83.82" x2="195.58" y2="83.82" width="0.1524" layer="91"/>
+</segment>
+</net>
+<net name="N$31" class="0">
+<segment>
+<pinref part="R40" gate="G$1" pin="1"/>
+<wire x1="198.12" y1="93.98" x2="200.66" y2="93.98" width="0.1524" layer="91"/>
 <pinref part="DAC2" gate="G$1" pin="VOUTA"/>
 <wire x1="195.58" y1="86.36" x2="198.12" y2="86.36" width="0.1524" layer="91"/>
 <wire x1="198.12" y1="86.36" x2="198.12" y2="93.98" width="0.1524" layer="91"/>
-<pinref part="R6" gate="G$1" pin="1"/>
-<wire x1="198.12" y1="93.98" x2="200.66" y2="93.98" width="0.1524" layer="91"/>
-</segment>
-</net>
-<net name="N$31" class="0">
-<segment>
-<pinref part="DAC2" gate="G$1" pin="VOUTB"/>
-<wire x1="195.58" y1="83.82" x2="198.12" y2="83.82" width="0.1524" layer="91"/>
-<wire x1="198.12" y1="83.82" x2="198.12" y2="78.74" width="0.1524" layer="91"/>
-<pinref part="R40" gate="G$1" pin="1"/>
-<wire x1="198.12" y1="78.74" x2="200.66" y2="78.74" width="0.1524" layer="91"/>
-</segment>
-</net>
+</segment>
+</net>

Commit message: intermediate
Connections:
- net N$10: now also IC2.2@RC; no longer IC2.1@RC
- net N$20: now also IC2.1@RC; no longer IC2.2@RC
Changed lines of the file:
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@@
 <wire x1="165.1" y1="83.82" x2="165.1" y2="106.68" width="0.1524" layer="91"/>
 <junction x="165.1" y="83.82"/>
-<wire x1="165.1" y1="83.82" x2="165.1" y2="71.12" width="0.1524" layer="91"/>
-<pinref part="IC2" gate="G$1" pin="2@RC"/>
-<wire x1="165.1" y1="71.12" x2="134.62" y2="71.12" width="0.1524" layer="91"/>
+<wire x1="165.1" y1="83.82" x2="165.1" y2="73.66" width="0.1524" layer="91"/>
+<pinref part="IC2" gate="G$1" pin="1@RC"/>
+<wire x1="165.1" y1="73.66" x2="134.62" y2="73.66" width="0.1524" layer="91"/>
 </segment>
 </net>
@@
 <segment>
 <pinref part="DAC2" gate="G$1" pin="SDI"/>
-<wire x1="134.62" y1="73.66" x2="167.64" y2="73.66" width="0.1524" layer="91"/>
 <wire x1="172.72" y1="81.28" x2="167.64" y2="81.28" width="0.1524" layer="91"/>
 <wire x1="167.64" y1="81.28" x2="167.64" y2="104.14" width="0.1524" layer="91"/>
@@
 <wire x1="167.64" y1="104.14" x2="172.72" y2="104.14" width="0.1524" layer="91"/>
 <junction x="167.64" y="81.28"/>
-<wire x1="167.64" y1="73.66" x2="167.64" y2="81.28" width="0.1524" layer="91"/>
-<pinref part="IC2" gate="G$1" pin="1@RC"/>
+<wire x1="167.64" y1="71.12" x2="167.64" y2="81.28" width="0.1524" layer="91"/>
+<pinref part="IC2" gate="G$1" pin="2@RC"/>
+<wire x1="167.64" y1="71.12" x2="134.62" y2="71.12" width="0.1524" layer="91"/>
 </segment>
 </net>
